Commit message: Update Obstacle Avoidance

File: install/TeleARM/share/TeleARM/urdf/telearm.urdf.xacro (robot description, xacro)
@@ -151,5 +151,5 @@
   <joint name="body_to_lidar_link" type="fixed">
     <!-- Front license-plate area (body mesh: x front~2.19, z roof~1.18, z bottom~0) -->
-    <origin xyz="0 0 0.5" rpy="0 0 0"/>
+    <origin xyz="2.1 0 0.9" rpy="0 0 0"/>
     <parent link="body"/>
     <child link="lidar_link"/>
